File: modular-bridge/cdf-modular-bridge-rev2.brd (EAGLE design)
At the start: 50.8 x 94 mm, 21 parts, among them Q1 Ixgh48n60a3, Q2 Ixgh48n60a3, T1 PULSE-P0584NL

Commit message: small changes
Parts:
- removed C1: PEH534YDC3220M2, rcl:EB35D
- added TP3, TP4: PTR1PAD1-17, testpad:P1-17
Connections:
- net DC+: now also TP4.TP; no longer C1.+
- net DC-: now also TP3.TP; no longer C1.-
Other:
- board size 50.8 x 94 mm -> 50.8 x 53.3 mm
- board text removed: "READD tSTOP LAYER!!!"
Changed lines of the file:
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@@
 <setting verticaltext="up"/>
 </settings>
-<grid distance="100" unitdist="mil" unit="mil" style="lines" multiple="1" display="yes" altdistance="0.025" altunitdist="inch" altunit="inch"/>
+<grid distance="10" unitdist="mil" unit="mil" style="lines" multiple="1" display="yes" altdistance="0.025" altunitdist="inch" altunit="inch"/>
 <layers>
 <layer number="1" name="Top" color="4" fill="1" visible="yes" active="yes"/>
@@
 <layer number="25" name="tNames" color="7" fill="1" visible="yes" active="yes"/>
 <layer number="26" name="bNames" color="7" fill="1" visible="yes" active="yes"/>
-<layer number="27" name="tValues" color="7" fill="1" visible="yes" active="yes"/>
-<layer number="28" name="bValues" color="7" fill="1" visible="yes" active="yes"/>
-<layer number="29" name="tStop" color="7" fill="3" visible="no" active="yes"/>
+<layer number="27" name="tValues" color="7" fill="1" visible="no" active="yes"/>
+<layer number="28" name="bValues" color="7" fill="1" visible="no" active="yes"/>
+<layer number="29" name="tStop" color="7" fill="3" visible="yes" active="yes"/>
 <layer number="30" name="bStop" color="7" fill="6" visible="no" active="yes"/>
 <layer number="31" name="tCream" color="7" fill="4" visible="no" active="yes"/>
@@
 <board>
 <plain>
-<wire x1="0" y1="-40.64" x2="50.8" y2="-40.64" width="0" layer="20"/>
-<wire x1="50.8" y1="-40.64" x2="50.8" y2="53.34" width="0" layer="20"/>
+<wire x1="0" y1="0" x2="50.8" y2="0" width="0" layer="20"/>
+<wire x1="50.8" y1="0" x2="50.8" y2="53.34" width="0" layer="20"/>
 <wire x1="50.8" y1="53.34" x2="0" y2="53.34" width="0" layer="20"/>
-<wire x1="0" y1="53.34" x2="0" y2="-40.64" width="0" layer="20"/>
+<wire x1="0" y1="53.34" x2="0" y2="0" width="0" layer="20"/>
 <text x="0.762" y="9.5504" size="5.08" layer="21" font="vector">+</text>
-<text x="46.736" y="0.254" size="5.08" layer="21" font="vector">-</text>
+<text x="46.228" y="10.922" size="5.08" layer="21" font="vector">-</text>
 <text x="31.115" y="3.4544" size="1.016" layer="21" font="vector" rot="R180">CDF MoBridge
 rev 2</text>
@@
 <vertex x="50.546" y="51.2064"/>
 </polygon>
-<text x="57.912" y="58.166" size="1.778" layer="21">READD tSTOP LAYER!!!</text>
 </plain>
 <attributes>
@@
 <element name="D4" library="keves" package="TPSMB15CA" value="TPSMB30CA" x="45.466" y="41.9354" rot="MR180"/>
 <element name="T1" library="keves" package="PULSE-P0584NL" value="PULSE-P0584NL" x="25.4" y="18.1864" rot="R90"/>
-<element name="X1" library="con-ptr500" package="AK500/2" value="" x="12.7" y="2.4384">
+<element name="X1" library="con-ptr500" package="AK500/2" value="" x="12.7" y="2.4384" smashed="yes">
 <attribute name="MPN" value="" x="12.7" y="2.4384" size="1.778" layer="27" display="off"/>
 <attribute name="OC_NEWARK" value="unknown" x="12.7" y="2.4384" size="1.778" layer="27" display="off"/>
 <attribute name="OC_FARNELL" value="unknown" x="12.7" y="2.4384" size="1.778" layer="27" display="off"/>
 <attribute name="MF" value="" x="12.7" y="2.4384" size="1.778" layer="27" display="off"/>
+<attribute name="VALUE" x="7.62" y="-3.2766" size="1.778" layer="27" ratio="10"/>
 </element>
 <element name="OUT" library="keves" package="BIG-ASS-HOLE" value="BIG-ASS-HOLE" x="25.4" y="46.8884"/>
 <element name="DC+" library="keves" package="BIG-ASS-HOLE" value="BIG-ASS-HOLE" x="12.7" y="15.1384"/>
 <element name="DC-" library="keves" package="BIG-ASS-HOLE" value="BIG-ASS-HOLE" x="38.1" y="15.1384"/>
-<element name="X2" library="con-ptr500" package="AK500/2" value="" x="38.1" y="2.4384">
+<element name="X2" library="con-ptr500" package="AK500/2" value="" x="38.1" y="2.4384" smashed="yes">
 <attribute name="OC_FARNELL" value="unknown" x="38.1" y="2.4384" size="1.778" layer="27" display="off"/>
 <attribute name="OC_NEWARK" value="unknown" x="38.1" y="2.4384" size="1.778" layer="27" display="off"/>
 <attribute name="MPN" value="" x="38.1" y="2.4384" size="1.778" layer="27" display="off"/>
 <attribute name="MF" value="" x="38.1" y="2.4384" size="1.778" layer="27" display="off"/>
-</element>
-<element name="TP1" library="testpad" package="P1-17" value="PTR1PAD1-17" x="2.54" y="2.4384" smashed="yes">
-<attribute name="TP_SIGNAL_NAME" value="" x="1.27" y="-0.7366" size="1" layer="37"/>
-<attribute name="VALUE" x="2.54" y="2.4384" size="0.0254" layer="27"/>
-</element>
-<element name="TP2" library="testpad" package="P1-17" value="PTR1PAD1-17" x="48.26" y="2.4384" smashed="yes">
-<attribute name="TP_SIGNAL_NAME" value="" x="46.99" y="-0.7366" size="1" layer="37"/>
-<attribute name="VALUE" x="48.26" y="2.4384" size="0.0254" layer="27"/>
+<attribute name="VALUE" x="33.02" y="-3.2766" size="1.778" layer="27" ratio="10"/>
+</element>
+<element name="TP1" library="testpad" package="P1-17" value="PTR1PAD1-17" x="2.54" y="2.413" smashed="yes">
+<attribute name="TP_SIGNAL_NAME" value="" x="1.27" y="-0.762" size="1" layer="37"/>
+<attribute name="VALUE" x="2.54" y="2.413" size="0.0254" layer="27"/>
+</element>
+<element name="TP2" library="testpad" package="P1-17" value="PTR1PAD1-17" x="48.26" y="2.413" smashed="yes">
+<attribute name="TP_SIGNAL_NAME" value="" x="46.99" y="-0.762" size="1" layer="37"/>
+<attribute name="VALUE" x="48.26" y="2.413" size="0.0254" layer="27"/>
 </element>
 <element name="D5" library="keves" package="TO220ABS" value="FMN-2206S" x="17.399" y="35.179" rot="R90"/>
-<element name="D7" library="keves" package="TO220ABS" value="FMN-2206S" x="16.51" y="35.179" rot="R270"/>
+<element name="D7" library="keves" package="TO220ABS" value="FMN-2206S" x="16.51" y="35.179" smashed="yes" rot="R270">
+<attribute name="NAME" x="10.4648" y="31.877" size="1.27" layer="25" ratio="10" rot="R270"/>
+<attribute name="VALUE" x="8.89" y="40.259" size="1.27" layer="27" ratio="10" rot="R270"/>
+</element>
 <element name="D6" library="keves" package="TO220ABS" value="FMN-2206S" x="39.624" y="29.591"/>
 <element name="D8" library="keves" package="TO220ABS" value="FMN-2206S" x="39.624" y="30.607" rot="R180"/>
-<element name="C1" library="rcl" package="EB35D" value="PEH534YDC3220M2" x="24.765" y="-20.955"/>
+<element name="TP3" library="testpad" package="P1-17" value="PTR1PAD1-17" x="45.212" y="2.413" smashed="yes">
+<attribute name="TP_SIGNAL_NAME" value="" x="43.942" y="-0.762" size="1" layer="37"/>
+<attribute name="VALUE" x="45.212" y="2.413" size="0.0254" layer="27"/>
+</element>
+<element name="TP4" library="testpad" package="P1-17" value="PTR1PAD1-17" x="5.842" y="2.413" smashed="yes">
+<attribute name="TP_SIGNAL_NAME" value="" x="4.572" y="-0.762" size="1" layer="37"/>
+<attribute name="VALUE" x="5.842" y="2.413" size="0.0254" layer="27"/>
+</element>
 </elements>
 <signals>
@@
 <wire x1="37.846" y1="15.3924" x2="38.1" y2="15.1384" width="1.778" layer="1"/>
 <contactref element="TP2" pad="TP"/>
-<wire x1="48.26" y1="2.4384" x2="48.26" y2="9.8044" width="2.54" layer="1"/>
+<wire x1="48.26" y1="2.413" x2="48.26" y2="9.8044" width="2.54" layer="1"/>
 <contactref element="DC-" pad="X@1"/>
 <contactref element="DC-" pad="X@2"/>
@@
 <wire x1="47.9044" y1="41.9354" x2="47.9044" y2="47.854" width="1.778" layer="16"/>
 <wire x1="47.9044" y1="47.854" x2="47.36" y2="48.3984" width="1.778" layer="16"/>
-<contactref element="C1" pad="-"/>
-<wire x1="48.26" y1="2.4384" x2="29.845" y2="-20.955" width="0" layer="19" extent="1-1"/>
+<contactref element="TP3" pad="TP"/>
+<polygon width="0.4064" layer="1" thermals="no">
+<vertex x="49.276" y="8.636"/>
+<vertex x="43.18" y="8.636"/>
+<vertex x="43.18" y="0.508"/>
+<vertex x="49.276" y="0.508"/>
+</polygon>
 </signal>
 <signal name="N$7">
@@
 </polygon>
 <contactref element="TP1" pad="TP"/>
-<wire x1="2.54" y1="2.4384" x2="2.54" y2="6.5024" width="2.54" layer="1"/>
+<wire x1="2.54" y1="2.413" x2="2.54" y2="6.5024" width="2.54" layer="1"/>
 <wire x1="2.54" y1="6.5024" x2="6.858" y2="10.8204" width="2.54" layer="1"/>
 <contactref element="DC+" pad="X@1"/>
@@
 <wire x1="13.97" y1="35.179" x2="9.271" y2="35.179" width="1.778" layer="1"/>
 <wire x1="9.271" y1="35.179" x2="8.89" y2="35.56" width="1.778" layer="1"/>
-<contactref element="C1" pad="+"/>
-<wire x1="2.54" y1="2.4384" x2="19.685" y2="-20.955" width="0" layer="19" extent="1-1"/>
+<contactref element="TP4" pad="TP"/>
+<polygon width="0.4064" layer="1" thermals="no">
+<vertex x="7.874" y="8.89"/>
+<vertex x="7.874" y="0.762"/>
+<vertex x="1.27" y="0.762"/>
+<vertex x="1.27" y="7.366"/>
+<vertex x="6.604" y="12.7"/>
+<vertex x="7.874" y="12.7"/>
+<vertex x="7.874" y="9.144"/>
+</polygon>
 </signal>
 <signal name="N$1">
