File: modular-bridge/cdf-modular-bridge-rev2.sch (EAGLE design)
At the start: 21 parts, among them Q1 Ixgh48n60a3, Q2 Ixgh48n60a3, T1 PULSE-P0584NL

Commit message: small changes
Parts:
- removed C1: PEH534YDC3220M2, rcl:CPOL-EUE10-35
- added TP3, TP4: PTR1PAD1-17, testpad:PTR1PAD1-17
Connections:
- net DC+: now also TP4.TP; no longer C1.+
- net DC-: now also TP3.TP; no longer C1.-
Other:
- note removed: "10mm lead spacing, 35mm outer diameter"
Changed lines of the file:
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@@
 <part name="D6" library="keves" deviceset="FMN-2206S" device=""/>
 <part name="D8" library="keves" deviceset="FMN-2206S" device=""/>
-<part name="C1" library="rcl" deviceset="CPOL-EU" device="E10-35" value="PEH534YDC3220M2"/>
+<part name="TP3" library="testpad" deviceset="PTR1" device="PAD1-17"/>
+<part name="TP4" library="testpad" deviceset="PTR1" device="PAD1-17"/>
 </parts>
 <sheets>
 <sheet>
 <plain>
-<text x="93.98" y="93.98" size="1.778" layer="97">For capacitor: 940C30S68K-F</text>
-<text x="154.94" y="35.56" size="1.778" layer="97" rot="R90">10mm lead spacing, 35mm outer diameter
-</text>
+<text x="93.98" y="101.6" size="1.778" layer="97">For capacitor: 940C30S68K-F</text>
 </plain>
 <instances>
@@
 <instance part="D6" gate="1" x="86.36" y="40.64"/>
 <instance part="D8" gate="1" x="101.6" y="40.64"/>
-<instance part="C1" gate="G$1" x="142.24" y="58.42" smashed="yes">
-<attribute name="NAME" x="143.383" y="58.9026" size="1.778" layer="95"/>
-<attribute name="VALUE" x="149.3774" y="54.483" size="1.778" layer="96" rot="R90"/>
-</instance>
+<instance part="TP3" gate="G$1" x="91.44" y="15.24" rot="R90"/>
+<instance part="TP4" gate="G$1" x="91.44" y="96.52" rot="R90"/>
 </instances>
 <busses>
@@
 <wire x1="60.96" y1="20.32" x2="22.86" y2="20.32" width="0.1524" layer="91"/>
 <junction x="60.96" y="20.32"/>
-<wire x1="73.66" y1="20.32" x2="73.66" y2="10.16" width="0.1524" layer="91"/>
+<wire x1="73.66" y1="20.32" x2="73.66" y2="15.24" width="0.1524" layer="91"/>
 <junction x="73.66" y="20.32"/>
 <pinref part="DC-" gate="G$1" pin="P$1"/>
-<wire x1="73.66" y1="10.16" x2="73.66" y2="2.54" width="0.1524" layer="91"/>
+<wire x1="73.66" y1="15.24" x2="73.66" y2="2.54" width="0.1524" layer="91"/>
 <wire x1="88.9" y1="20.32" x2="73.66" y2="20.32" width="0.1524" layer="91"/>
 <pinref part="T1" gate="G$1" pin="SEC2_POS"/>
@@
 <junction x="91.44" y="27.94"/>
 <junction x="96.52" y="27.94"/>
-<pinref part="C1" gate="G$1" pin="-"/>
-<wire x1="142.24" y1="53.34" x2="142.24" y2="10.16" width="0.1524" layer="91"/>
-<wire x1="142.24" y1="10.16" x2="73.66" y2="10.16" width="0.1524" layer="91"/>
+<pinref part="TP3" gate="G$1" pin="TP"/>
+<wire x1="88.9" y1="15.24" x2="73.66" y2="15.24" width="0.1524" layer="91"/>
+<junction x="73.66" y="15.24"/>
 </segment>
 </net>
@@
 <pinref part="DC+" gate="G$1" pin="P$1"/>
 <wire x1="73.66" y1="88.9" x2="73.66" y2="91.44" width="0.1524" layer="91"/>
-<wire x1="73.66" y1="91.44" x2="73.66" y2="101.6" width="0.1524" layer="91"/>
-<wire x1="73.66" y1="101.6" x2="73.66" y2="106.68" width="0.1524" layer="91"/>
+<wire x1="73.66" y1="91.44" x2="73.66" y2="96.52" width="0.1524" layer="91"/>
+<wire x1="73.66" y1="96.52" x2="73.66" y2="106.68" width="0.1524" layer="91"/>
 <wire x1="88.9" y1="91.44" x2="73.66" y2="91.44" width="0.1524" layer="91"/>
 <junction x="73.66" y="91.44"/>
@@
 <junction x="86.36" y="88.9"/>
 <junction x="73.66" y="88.9"/>
-<pinref part="C1" gate="G$1" pin="+"/>
-<wire x1="142.24" y1="60.96" x2="142.24" y2="101.6" width="0.1524" layer="91"/>
-<wire x1="142.24" y1="101.6" x2="73.66" y2="101.6" width="0.1524" layer="91"/>
-<junction x="73.66" y="101.6"/>
+<pinref part="TP4" gate="G$1" pin="TP"/>
+<wire x1="88.9" y1="96.52" x2="73.66" y2="96.52" width="0.1524" layer="91"/>
+<junction x="73.66" y="96.52"/>
 </segment>
 </net>
@@
 </schematic>
 </drawing>
-<compatibility>
-<note version="6.3" minversion="6.2.2" severity="warning">
-Since Version 6.2.2 text objects can contain more than one line,
-which will not be processed correctly with this version.
-</note>
-</compatibility>
 </eagle>
